File: dummyvideo.brd (EAGLE design)
At the start: 18.7 x 32.4 mm, 17 parts, among them IC1 NE555SO

Commit message: Final Board revision
Parts:
- moved PWR_PAD_VCC 1.27 mm to (16.5, 10.8)
Routing:
- net VCC: track 13.6 -> 14.2 mm
Changed lines of the file:
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@@
 <setting verticaltext="up"/>
 </settings>
-<grid distance="1" unitdist="mil" unit="mil" style="lines" multiple="1" display="no" altdistance="0.025" altunitdist="inch" altunit="inch"/>
+<grid distance="0.05" unitdist="inch" unit="inch" style="lines" multiple="1" display="no" altdistance="0.025" altunitdist="inch" altunit="inch"/>
 <layers>
 <layer number="1" name="Top" color="4" fill="1" visible="yes" active="yes"/>
@@
 <layer number="42" name="bRestrict" color="1" fill="10" visible="no" active="yes"/>
 <layer number="43" name="vRestrict" color="2" fill="10" visible="no" active="yes"/>
-<layer number="44" name="Drills" color="7" fill="1" visible="no" active="yes"/>
+<layer number="44" name="Drills" color="7" fill="1" visible="yes" active="yes"/>
 <layer number="45" name="Holes" color="7" fill="1" visible="yes" active="yes"/>
 <layer number="46" name="Milling" color="3" fill="1" visible="no" active="yes"/>
@@
 <element name="JP_PAD1" library="wirepad" package="SMD1,27-2,54" value="" x="6.35" y="1.905"/>
 <element name="JP_PAD2" library="wirepad" package="SMD1,27-2,54" value="" x="8.255" y="1.905"/>
-<element name="PWR_PAD_VCC" library="wirepad" package="SMD1,27-2,54" value="" x="16.51" y="9.525" rot="R90"/>
+<element name="PWR_PAD_VCC" library="wirepad" package="SMD1,27-2,54" value="" x="16.51" y="10.795" rot="R90"/>
 <element name="PWR_PAD_GND" library="wirepad" package="SMD1,27-2,54" value="" x="16.51" y="12.7" rot="R90"/>
 <element name="PAD_Y" library="wirepad" package="SMD1,27-2,54" value="" x="16.51" y="27.305" rot="R90"/>
@@
 <contactref element="JP_PAD2" pad="1"/>
 <contactref element="PWR_PAD_VCC" pad="1"/>
-<wire x1="16.51" y1="9.525" x2="12.065" y2="9.525" width="0.4064" layer="1"/>
-<wire x1="12.065" y1="9.525" x2="8.255" y2="5.715" width="0.4064" layer="1"/>
+<wire x1="16.51" y1="10.795" x2="13.335" y2="10.795" width="0.4064" layer="1"/>
+<wire x1="13.335" y1="10.795" x2="8.255" y2="5.715" width="0.4064" layer="1"/>
 <wire x1="8.255" y1="5.715" x2="8.255" y2="1.905" width="0.4064" layer="1"/>
 </signal>

Commit message: Spannungsteiler war zu hochohmig -> angepasst
Parts:
- R3: value 4,7K -> 470R
- R4: value 1,5K -> 150R
Changed lines of the file:
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@@
 <element name="C1" library="resistor" package="C0805" value="10n" x="4.445" y="20.955" rot="R90"/>
 <element name="D1" library="n39" package="SOD80C" value="1N4148SOD-80" x="13.335" y="19.05" rot="R270"/>
-<element name="R3" library="resistor" package="R0805" value="4,7K" x="10.16" y="26.035" rot="R270"/>
-<element name="R4" library="resistor" package="R0805" value="1,5K" x="12.7" y="26.035" rot="R90"/>
+<element name="R3" library="resistor" package="R0805" value="470R" x="10.16" y="26.035" rot="R270"/>
+<element name="R4" library="resistor" package="R0805" value="150R" x="12.7" y="26.035" rot="R90"/>
 <element name="LED1" library="led" package="CHIP-LED0603" value="gn LC" x="2.54" y="6.35"/>
 <element name="R5" library="resistor" package="R0805" value="1,5K" x="2.54" y="3.175" rot="R270"/>
